File: G64-A00.kicad_pcb (KiCad board)
At the start: 2 copper layers, 390 x 179.8 mm, 227 parts, among them CN1 KEYBOARD_20PIN_MALE, CN10 LED_CONNECTOR, CN2 USER_PORT_CON, CN3 CASSETTE_PORT_CON, CN4 SERIAL_BUS_CON, CN5 AV_CONN, CN6 EXPANSION_PORT, CN7 POWER_CON, CN8 CONTROL_PORT, CN9 CONTROL_PORT, M1 MODULATOR_LONGBOARD, Q1 2SC1815, Q2 2SC1815, Q3 TP29B/2SD880, Q7 2SC1815, Q8 2SC1815, SW1 POWER_SWITCH, U1 CIA_U1, U10 4164-2, U11 4164-2, U12 4164-2, U13 74LS257, U14 74LS258, U15 74LS139, U16 4066_U28, U17 PLA_U17, U18 6581, U19 VIC, U2 CIA_U2, U20 556, U21 4164-2, U22 4164-2, U23 4164-2, U24 4164-2, U25 74LS257, U26 74LS373, U27 7408_U27, U28 4066_U28, U29 74LS74, U3 2364A, U30 74LS193, U31 74LS629N, U32 MC4044, U4 2364A, U5 2332A, U6 2114, U7 6510_MPU, U8 7406N, U9 4164-2, Y1 Crystal

Commit message: change vias to 0.4/0.9 add netclass for power and clocks
Parts:
- C38: value 51pF -> 4.7nF
Connections:
- net /'9VAC~~ renamed /9VAC'
- net /250407_sheet2/AEC renamed /G64-A00_sheet2/AEC
- net /250407_sheet2/AUDIO_IN renamed /G64-A00_sheet2/AUDIO_IN
- net /250407_sheet2/AUDIO_OUT renamed /G64-A00_sheet2/AUDIO_OUT
- net /250407_sheet2/BA renamed /G64-A00_sheet2/BA
- net /250407_sheet2/CHROMA renamed /G64-A00_sheet2/CHROMA
- net /250407_sheet2/CHROMA_O renamed /G64-A00_sheet2/CHROMA_O
- net /250407_sheet2/COMP_O renamed /G64-A00_sheet2/COMP_O
- net /250407_sheet2/GR\~W~ renamed /G64-A00_sheet2/GR\~W~
- net /250407_sheet2/LUMA renamed /G64-A00_sheet2/LUMA
- net /250407_sheet2/LUMA_O renamed /G64-A00_sheet2/LUMA_O
- net /250407_sheet2/MA0 renamed /G64-A00_sheet2/MA0
- net /250407_sheet2/MA1 renamed /G64-A00_sheet2/MA1
- net /250407_sheet2/MA2 renamed /G64-A00_sheet2/MA2
- net /250407_sheet2/MA3 renamed /G64-A00_sheet2/MA3
- net /250407_sheet2/MA4 renamed /G64-A00_sheet2/MA4
- net /250407_sheet2/MA5 renamed /G64-A00_sheet2/MA5
- net /250407_sheet2/MA6 renamed /G64-A00_sheet2/MA6
- net /250407_sheet2/MA7 renamed /G64-A00_sheet2/MA7
- net /250407_sheet2/VA0 renamed /G64-A00_sheet2/VA0
- net /250407_sheet2/VA1 renamed /G64-A00_sheet2/VA1
- net /250407_sheet2/VA2 renamed /G64-A00_sheet2/VA2
- net /250407_sheet2/VA3 renamed /G64-A00_sheet2/VA3
- net /250407_sheet2/VA4 renamed /G64-A00_sheet2/VA4
- net /250407_sheet2/VA5 renamed /G64-A00_sheet2/VA5
- net /250407_sheet2/VA6 renamed /G64-A00_sheet2/VA6
- net /250407_sheet2/VA6' renamed /G64-A00_sheet2/VA6'
- net /250407_sheet2/VA7 renamed /G64-A00_sheet2/VA7
- net /250407_sheet2/VA7' renamed /G64-A00_sheet2/VA7'
- net /250407_sheet2/~AEC~ renamed /G64-A00_sheet2/~AEC~
- net /250407_sheet2/~BASIC~ renamed /G64-A00_sheet2/~BASIC~
- net /250407_sheet2/~CASRAM~ renamed /G64-A00_sheet2/~CASRAM~
- net /250407_sheet2/~CASRAM~' renamed /G64-A00_sheet2/~CASRAM~'
- net /250407_sheet2/~CAS~ renamed /G64-A00_sheet2/~CAS~
- net /250407_sheet2/~CHAROM~ renamed /G64-A00_sheet2/~CHAROM~
- net /250407_sheet2/~CIAS~ renamed /G64-A00_sheet2/~CIAS~
- net /250407_sheet2/~COLOR~ renamed /G64-A00_sheet2/~COLOR~
- net /250407_sheet2/~DMA~ renamed /G64-A00_sheet2/~DMA~
- net /250407_sheet2/~EXROM~ renamed /G64-A00_sheet2/~EXROM~
- net /250407_sheet2/~GAME~ renamed /G64-A00_sheet2/~GAME~
- net /250407_sheet2/~I\O~ renamed /G64-A00_sheet2/~I\O~
- net /250407_sheet2/~KERNAL renamed /G64-A00_sheet2/~KERNAL
- net /250407_sheet2/~RAS~ renamed /G64-A00_sheet2/~RAS~
- net /250407_sheet2/~RESET'~ renamed /G64-A00_sheet2/~RESET'~
- net /250407_sheet2/~ROMH~ renamed /G64-A00_sheet2/~ROMH~
- net /250407_sheet2/~ROML~ renamed /G64-A00_sheet2/~ROML~
- net /250407_sheet2/~SID~ renamed /G64-A00_sheet2/~SID~
- net /250407_sheet2/~VIC~ renamed /G64-A00_sheet2/~VIC~
- net Net-(C101-Pad1) renamed /G64-A00_sheet2/VIC_VCC
- net Net-(C20-Pad1) renamed /9V_IN'
- net Net-(C21-Pad1) renamed /9V_F
- net Net-(C50-Pad1) renamed /G64-A00_sheet2/SID_VCC
- net Net-(C51-Pad1) renamed /G64-A00_sheet2/SID_VDD
- net Net-(C54-Pad1) renamed /G64-A00_sheet2/VIC_VDD
- net Net-(C97-Pad2) renamed /5V_IN
- C20 pad 2: /9VAC -> /9V_IN
- C21 pad 2: /9VAC~~ -> /9VAC
- C90 pad 2: /9VAC~~ -> /9VAC
- C99 pad 2: /9VAC~~ -> /9VAC
- CN2 pad 10: /9VAC~~ -> /9VAC
- CR4 pad 4: /9VAC~~ -> /9VAC
- L4 pad 3: /9VAC -> /9V_IN
- L4 pad 4: /9VAC~~ -> /9VAC
- R5 pad 1: /9VAC~~ -> /9VAC
- SW1 pad 1: /9VAC -> /9V_IN
Routing:
- net /9VAC~~: track 527.5 -> 0.00 mm, vias 4 -> 0
- net /9VAC: track 47.2 -> 527.5 mm, vias 0 -> 4
- net /9V_IN: track 0.00 -> 47.2 mm
- net CAN+5V: track 298.9 -> 291.3 mm, vias 5 -> 3
- net (no net): track 88.6 -> 80.9 mm, vias 2 -> 0
- net Net-(U17-Pad1): track 7.40 -> 0.00 mm, vias 1 -> 0
- net GND: track 2396.8 -> 2393.0 mm, vias 83 -> 80
Other:
- net class CLK added: clearance 0.3, trace_width 0.25, via_dia 0.9, via_drill 0.4
- net class Default: via_dia 0.8 -> 0.9
- net class PWR added: clearance 0.25, trace_width 1.2, via_dia 0.9, via_drill 0.4

Commit message: update many components on the PCB
Parts:
- C1, C10, C100, C101, C103, C105, C11, C16, C18, C2, C200, C204, C205, C22, C25, C26, C27, C28, C29, C3, C30, C31, C32, C33, C37, C39, C4, C40, C41, C42, C43, C44, C45, C46, C47, C48, C49, C5, C50, C51, C52, C53, C54, C56, C59, C6, C60, C66, C67, C68, C7, C74, C82, C84, C85, C89, C9, C92, C93, C95, C96, C97, C98, C99: footprint C64-pcb-library:CAP_P5.08mm -> pth_c:C_film_7x2.5
- C102, C107, C108, C12, C13, C14, C15, C17, C24, C34, C57, C62, C65, C8, C94: footprint C64-pcb-library:CAP_ELYT_RADIAL_P5.08mm_SMALL_RING -> pth_cp:CP_5p2x11
- C19, C88, C90: footprint C64-pcb-library:LARGE_ELECTROLYTIC_AXIAL_TH -> pth_cp:CP_10p5x20
- C20, C21: footprint C64-pcb-library:CAP_POLY_100V_TH_P5.08_and_P12.07mm -> pth_c:C_film_7x2.5
- C91: footprint C64-pcb-library:CAP_ELYT_RADIAL_P5.08mm -> pth_cp:CP_5p2x11
- R1, R100, R16, R17, R19, R2, R26, R28, R29, R3, R30, R31, R33, R34, R35, R36, R37, R38, R39, R4, R41, R42, R43, R44, R45, R5, R50, R51, R52, R53, R6, R7: footprint C64-pcb-library:RESISTOR -> pth_r:r_0250p12_7
- RP1, RP2, RP3: footprint C64-pcb-library:RP_ARRAY_7WAY -> pth_r:rpak_sil_8
- RP4: footprint C64-pcb-library:RP_ARRAY_9WAY -> pth_r:rpak_sil_10
- U1, U19, U2, U7: footprint C64-pcb-library:DIP40 -> pth_dil:DIP-40_600
- U10, U11, U12, U13, U14, U15, U21, U22, U23, U24, U25, U30, U31, U9: footprint C64-pcb-library:DIP16 -> pth_dil:DIP-16_300
- U16, U20, U27, U28, U29, U32, U8: footprint C64-pcb-library:DIP14 -> pth_dil:DIP-14_300
- U17, U18: footprint C64-pcb-library:DIP28 -> pth_dil:DIP-28_600
- U26: footprint C64-pcb-library:DIP20 -> pth_dil:DIP-20_300
- U3, U4, U5: footprint C64-pcb-library:DIP24 -> pth_dil:DIP-24_600
- U6: footprint C64-pcb-library:DIP18 -> pth_dil:DIP-18_300
- moved C19 27.6 mm to (368.3, 163.8)
- moved CR6 18.8 mm to (350.5, 173.4)
- moved C88 16.4 mm to (337.8, 163.8)
- moved C99 16.1 mm to (358.1, 133.3), turned to 270 degrees
- moved C90 15.5 mm to (353.1, 163.8)
- moved CR5 15.2 mm to (345.4, 173.4)
- moved RP4 11.4 mm to (317.5, 97.0)
- moved RP1 8.89 mm to (108.0, 161.9)
- moved RP2 8.89 mm to (108.0, 200.0)
- moved RP3 8.89 mm to (71.1, 66.7)
- moved R35 6.67 mm to (29.2, 208.9)
- moved R17 6.35 mm to (311.1, 141.6)
- moved R19 6.35 mm to (307.3, 141.6)
- moved R39 6.35 mm to (386.1, 208.9)
- moved R1 6.35 mm to (88.9, 75.6)
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Routing:
- net +5V: track 2212.9 -> 2256.0 mm
- net Net-(C90-Pad1): track 62.4 -> 23.7 mm
- net +9V_UNREG: track 491.9 -> 517.6 mm
- net Net-(C88-Pad1): track 73.1 -> 58.1 mm
- net /9V_IN: track 47.2 -> 35.7 mm
- net /+Vc: track 266.8 -> 275.4 mm
- net /9VAC: track 527.5 -> 533.4 mm, vias 4 -> 5
- net /G64-A00_sheet2/AEC: track 333.1 -> 328.2 mm
- net +12V: track 288.5 -> 293.0 mm
- net CAN+5V: track 291.3 -> 295.6 mm
- net /G64-A00_sheet2/VA6': track 132.2 -> 128.1 mm, vias 4 -> 2
- net /G64-A00_sheet2/~RAS~: track 366.8 -> 370.2 mm
- net Net-(C108-Pad1): track 19.5 -> 17.1 mm
- net Net-(C24-Pad1): track 30.6 -> 28.8 mm
- net Net-(C13-Pad1): track 36.8 -> 35.3 mm
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- removed copper zone on B.Cu, net (none)
- removed copper zone on F.Cu, net +5V
- removed copper zone on F.Cu, net /+Vc
- removed copper zone on B.Cu, net CAN+5V
- removed copper zone on F.Cu, net CAN+5V
Other:
- net class CLK: trace_width 0.25 -> 0.3
- net class Default: trace_width 0.25 -> 0.3

Commit message: add protection diodes to PCB
Parts:
- added CR100: D_Small_ALT, C64-pcb-library:RECTIFIER_TH_P12.7mm, F.Cu at (35.6, 148.0)
- added CR101: D_Small_ALT, C64-pcb-library:RECTIFIER_TH_P12.7mm, F.Cu at (35.6, 153.0)
- added CR102: D_Small_ALT, C64-pcb-library:RECTIFIER_TH_P12.7mm, F.Cu at (35.6, 170.8)
- added CR103: D_Small_ALT, C64-pcb-library:RECTIFIER_TH_P12.7mm, F.Cu at (35.6, 165.7)
- moved R50 5.72 mm to (29.2, 176.5)
- moved F1 2.54 mm to (374.6, 120.0)
- moved R30 2.54 mm to (29.2, 168.3)
Routing:
- net GND: track 2394.4 -> 2371.2 mm
- net +5V: track 2256.0 -> 2274.6 mm, vias 28 -> 30
- net +9V_UNREG: track 517.6 -> 500.1 mm
- net /CLK': track 102.7 -> 118.9 mm
- net /DATA': track 78.7 -> 92.4 mm
- net /9V_F: track 67.7 -> 55.4 mm
- net /9VAC': track 434.0 -> 424.2 mm
- net /G64-A00_sheet2/VIC_VCC: track 40.3 -> 49.4 mm
- net CAN+5V: track 295.6 -> 287.3 mm, vias 3 -> 1
- net Net-(C105-Pad2): track 57.6 -> 53.1 mm
- net A11: track 541.3 -> 536.8 mm
- net A10: track 475.9 -> 471.4 mm
- net A9: track 488.8 -> 484.8 mm
- net A8: track 526.4 -> 522.6 mm
- net Net-(C13-Pad1): track 35.3 -> 37.8 mm
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
Commit message: change DIN footprints to accept both 5mm and 10mm retention add link to 3D models for a few footprints
Parts:
- CN10: footprint C64-pcb-library:LED_CON -> pin_strip:pin_strip_3
- moved CN10 2.54 mm to (397.5, 201.3), turned to 270 degrees
- moved CN5 0.06 mm to (211.6, 64.5)
Routing:
- net +5V: track 2274.6 -> 2307.5 mm
- net GND: track 2371.2 -> 2339.5 mm
- net +12V: track 293.0 -> 285.1 mm
- net +9V_UNREG: track 500.1 -> 492.9 mm
- net BTNA\~LP~: track 627.7 -> 620.8 mm
- net ~LORAM~: track 97.7 -> 94.9 mm
- net /G64-A00_sheet2/VA7: track 90.3 -> 89.1 mm
- net /CLK': track 118.9 -> 117.8 mm
- net ~NMI~: track 513.8 -> 512.9 mm
- net A15: track 370.7 -> 370.0 mm
- net /LED+: track 13.1 -> 12.6 mm
- net A0: track 533.1 -> 532.6 mm
