File: G64-A00.kicad_pcb (KiCad board)
At the start: 2 copper layers, 390 x 179.8 mm, 191 parts, among them CN1 KEYBOARD_20PIN_MALE, CN10 LED_CONNECTOR, CN2 USER_PORT_CON, CN3 CASSETTE_PORT_CON, CN4 SERIAL_BUS_CON, CN5 AV_CONN, CN6 EXPANSION_PORT, CN7 POWER_CON, CN8 CONTROL_PORT, CN9 CONTROL_PORT, M1 MODULATOR_LONGBOARD, Q1 2SC1815, Q2 2SC1815, Q3 TP29B/2SD880, Q8 2SC1815, SW1 POWER_SWITCH, U1 CIA_U1, U10 4164-2, U11 4164-2, U12 4164-2, U13 74LS257, U14 74LS258, U15 74LS139, U16 4066_U28, U17 PLA_U17, U18 6581, U19 VIC, U2 CIA_U2, U20 556, U21 4164-2, U22 4164-2, U23 4164-2, U24 4164-2, U25 74LS257, U26 74LS373, U27 7408_U27, U28 4066_U28, U3 2364A, U31 8701, U4 2364A, U5 2332A, U6 2114, U7 6510_MPU, U8 7406N, U9 4164-2, Y1 Crystal

Commit message: add extra protection diodes on IEC port
Parts:
- removed CR100, CR101, CR102, CR103: D_Small_ALT, C64-pcb-library:RECTIFIER_TH_P12.7mm
- added CR12: D_Small_ALT, C64-pcb-library:RECTIFIER_TH_P12.7mm, F.Cu at (123.2, 94.6)
- added CR13: D_Small_ALT, C64-pcb-library:RECTIFIER_TH_P12.7mm, F.Cu at (35.6, 148.0)
- added CR14: D_Small_ALT, C64-pcb-library:RECTIFIER_TH_P12.7mm, F.Cu at (35.6, 170.8)
- added CR15: D_Small_ALT, C64-pcb-library:RECTIFIER_TH_P12.7mm, F.Cu at (35.6, 153.0)
- added CR16: D_Small_ALT, C64-pcb-library:RECTIFIER_TH_P12.7mm, F.Cu at (35.6, 165.7)
- added CR9: D_Small_ALT, C64-pcb-library:RECTIFIER_TH_P12.7mm, F.Cu at (138.4, 94.6)
- moved C1 5.68 mm to (135.9, 89.5)
- moved C96 4.02 mm to (77.5, 75.6), turned to 0 degrees
- moved C18 2.54 mm to (113.0, 89.5)
Routing:
- net +5V: track 2391.9 -> 2367.4 mm, vias 31 -> 33
- net +12V: track 280.5 -> 291.2 mm
- net ~RESET~: track 625.2 -> 615.0 mm
- net /CASS_RD: track 271.9 -> 278.7 mm
- net A8: track 507.9 -> 502.5 mm
- net GND: track 2084.0 -> 2078.7 mm
- net D0: track 685.9 -> 680.7 mm
- net D7: track 488.1 -> 483.3 mm
- net D6: track 509.3 -> 504.5 mm
- net D5: track 497.3 -> 492.4 mm
- net D4: track 549.1 -> 544.2 mm
- net D3: track 587.2 -> 582.3 mm
- net D2: track 656.0 -> 651.2 mm
- net A6: track 527.8 -> 523.1 mm
- net D1: track 639.1 -> 634.4 mm
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